Commit message: tutorial files

File: 3rpr_description/urdf/05-visual.urdf (robot description, URDF)
Before this commit: robot visual, 16 links, 15 joints
Links:
- link left_gripper: geometry visual mesh filename=package://urdf_tutorial/meshes/l_finger.dae
- link left_tip: geometry visual mesh filename=package://urdf_tutorial/meshes/l_finger_tip.dae
- link right_gripper: geometry visual mesh filename=package://urdf_tutorial/meshes/l_finger.dae
- link right_tip: geometry visual mesh filename=package://urdf_tutorial/meshes/l_finger_tip.dae

File: 3rpr_description/urdf/06-flexible.urdf (robot description, URDF)
Before this commit: robot visual, 16 links, 15 joints
Links:
- link left_gripper: geometry visual mesh filename=package://urdf_tutorial/meshes/l_finger.dae
- link left_tip: geometry visual mesh filename=package://urdf_tutorial/meshes/l_finger_tip.dae
- link right_gripper: geometry visual mesh filename=package://urdf_tutorial/meshes/l_finger.dae
- link right_tip: geometry visual mesh filename=package://urdf_tutorial/meshes/l_finger_tip.dae
Joints:
- joint gripper_extension: limit (none) -> lower=-0.38 upper=0 effort=1000.0 velocity=0.5; type fixed -> prismatic
- joint head_swivel: axis (none) -> 0 0 1; type fixed -> continuous
- joint left_back_wheel_joint: axis (none) -> 0 1 0; type fixed -> continuous
- joint left_front_wheel_joint: axis (none) -> 0 1 0; type fixed -> continuous
- joint left_gripper_joint: axis (none) -> 0 0 1; limit (none) -> lower=0.0 upper=0.548 effort=1000.0 velocity=0.5; type fixed -> revolute
- joint right_back_wheel_joint: axis (none) -> 0 1 0; type fixed -> continuous
- joint right_front_wheel_joint: axis (none) -> 0 1 0; type fixed -> continuous
- joint right_gripper_joint: axis (none) -> 0 0 -1; limit (none) -> lower=0.0 upper=0.548 effort=1000.0 velocity=0.5; type fixed -> revolute
